File: Design/circuit design/_autosave-circuit design.kicad_pcb (KiCad board)
At the start: 2 copper layers, 18 parts, among them K1 R2_1A05, U1 STM32H7xx Dev Board, U2 ESP-01S, U3 HM-10, U4 uBlox_NEO_7M, U5 E-Paper_296x152_SSD1680, U6 MP1584EN, U7 EasyCard_IC, U8 TP4056

Commit message: [2026-03-13 10:18:17 From Windows 11 Home]: Windows auto commit
Parts:
- removed the REF** at (151.0, 136.1)
- removed the REF** at (151.0, 139.1)
Routing:
- net (no net): track 1096.7 -> 1056.7 mm
