File: Design/circuit design/_autosave-circuit design.kicad_pcb (KiCad board)
At the start: 2 copper layers, 16 parts, among them K1 R2_1A05, U1 STM32H7xx Dev Board, U2 ESP-01S, U3 HM-10, U4 uBlox_NEO_7M, U5 E-Paper_296x152_SSD1680, U6 MP1584EN, U7 EasyCard_IC, U8 TP4056

Commit message: [2026-03-13 11:18:16 From Windows 11 Home]: Windows auto commit
Parts:
- removed the REF** at (153.0, 144.1)
- removed the REF** at (153.0, 137.5)
- removed the REF** at (150.0, 144.0)
- removed the REF** at (153.0, 135.0)
- added ?: , , F.Cu at (150.0, 141.5)
- added ?: , , F.Cu at (153.0, 141.5)
- added ?: , , F.Cu at (150.0, 146.0)
- added ?: , , F.Cu at (153.0, 146.0)
- added ?: , , F.Cu at (150.5, 134.5)
- added ?: , , F.Cu at (150.5, 137.5)
- added REF**: TestPoint_Pad_D1.0mm, TestPoint:TestPoint_Pad_D1.0mm, F.Cu at (157.5, 134.5)
- added REF**: TestPoint_Pad_D1.0mm, TestPoint:TestPoint_Pad_D1.0mm, F.Cu at (148.0, 120.0)
- added REF**: TestPoint_Pad_D1.0mm, TestPoint:TestPoint_Pad_D1.0mm, F.Cu at (148.0, 122.5)
- added REF**: TestPoint_Pad_D1.0mm, TestPoint:TestPoint_Pad_D1.0mm, F.Cu at (152.0, 120.0)
- added REF**: TestPoint_Pad_D1.0mm, TestPoint:TestPoint_Pad_D1.0mm, F.Cu at (157.5, 137.5)
- added REF**: TestPoint_Pad_D1.0mm, TestPoint:TestPoint_Pad_D1.0mm, F.Cu at (152.0, 122.5)
Routing:
- net (no net): track 1053.6 -> 1052.9 mm

Commit message: [2026-03-13 11:48:16 From Windows 11 Home]: Windows auto commit
Parts:
- removed the REF** at (172.5, 111.6)
- removed the REF** at (172.4, 108.6)
- added ?: , , F.Cu at (170.0, 117.5)
- added ?: , , F.Cu at (170.0, 113.5)
- added ?: , , F.Cu at (176.0, 113.5)
- added ?: , , F.Cu at (176.0, 117.5)
- U1: footprint Module:MODULE_STM327H7xx Dev Module -> Module:MODULE_STM327H7xx Dev Module_1
- U2: footprint Connector_PinHeader_2.54mm:PinHeader_2x04_P2.54mm_Vertical -> Module:MODULE_ESP-01
- moved U2 13.8 mm to (128.5, 90.0), turned to 180 degrees
- moved REF** 1.00 mm to (153.0, 120.0)
- moved REF** 1.00 mm to (153.0, 122.5)
Routing:
- net (no net): track 1052.9 -> 1043.4 mm

Commit message: [2026-03-13 13:42:05 From Windows 11 Home]: Windows auto commit
Parts:
- moved REF** 1.00 mm to (147.0, 120.0)
- moved REF** 1.00 mm to (147.0, 122.5)
Routing:
- net (no net): track 1043.4 -> 1047.0 mm
Changed lines of the file:
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@@
 	(footprint "TestPoint:TestPoint_Pad_D1.0mm"
 		(layer "F.Cu")
-		(at 148 120)
+		(at 147 120)
 		(descr "SMD pad as test Point, diameter 1.0mm")
 		(tags "test point SMD pad")
@@
 	(footprint "TestPoint:TestPoint_Pad_D1.0mm"
 		(layer "F.Cu")
-		(at 148 122.5)
+		(at 147 122.5)
 		(descr "SMD pad as test Point, diameter 1.0mm")
 		(tags "test point SMD pad")
@@
 	)
 	(segment
-		(start 149 132.5)
-		(end 150 131.5)
-		(width 1)
-		(layer "F.Cu")
-		(net 0)
-	)
-	(segment
 		(start 157.5 137.5)
 		(end 164.5 137.5)
@@
 	)
 	(segment
-		(start 150 131.5)
-		(end 150 132.06)
-		(width 0.2)
-		(layer "F.Cu")
-		(net 0)
-	)
-	(segment
 		(start 145 94.5)
 		(end 145 96.88)
@@
 	)
 	(segment
-		(start 149.5 113.56)
-		(end 149.5 129.5)
-		(width 0.2)
-		(layer "F.Cu")
-		(net 0)
-	)
-	(segment
 		(start 172 105.56)
 		(end 172 140.56)
@@
 	)
 	(segment
-		(start 131.06 121.56)
-		(end 135.5 126)
+		(start 146.78 122.28)
+		(end 147 122.5)
 		(width 1)
 		(layer "F.Cu")
@@
 	)
 	(segment
-		(start 141.365002 143.194998)
-		(end 142.56 142)
-		(width 0.5)
+		(start 135.5 129)
+		(end 136.5 130)
+		(width 1)
 		(layer "F.Cu")
 		(net 0)
 	)
 	(segment
-		(start 149.5 129.5)
-		(end 149.5 130.06)
-		(width 0.2)
+		(start 135.5 132.5)
+		(end 149 132.5)
+		(width 1)
+		(layer "F.Cu")
+		(net 0)
+	)
+	(segment
+		(start 141.365002 143.194998)
+		(end 142.56 142)
+		(width 0.5)
 		(layer "F.Cu")
 		(net 0)
@@
 	)
 	(segment
+		(start 135.5 126)
+		(end 135.5 129)
+		(width 1)
+		(layer "F.Cu")
+		(net 0)
+	)
+	(segment
 		(start 148.5 143.56)
 		(end 147.25 144.81)
@@
 	)
 	(segment
-		(start 148.06 112.12)
-		(end 149.5 113.56)
-		(width 0.2)
-		(layer "F.Cu")
-		(net 0)
-	)
-	(segment
 		(start 155 151.06)
 		(end 156.605002 149.454998)
@@
 	)
 	(segment
-		(start 126 121.56)
-		(end 131.06 121.56)
-		(width 1)
-		(layer "F.Cu")
-		(net 0)
-	)
-	(segment
 		(start 146.5 145.06)
 		(end 144.5 147.06)
@@
 	)
 	(segment
-		(start 145 122.28)
-		(end 147.78 122.28)
+		(start 145 119.74)
+		(end 146.74 119.74)
 		(width 1)
 		(layer "F.Cu")
@@
 	)
 	(segment
-		(start 145 119.74)
-		(end 147.74 119.74)
-		(width 1)
-		(layer "F.Cu")
-		(net 0)
-	)
-	(segment
-		(start 130.1 124.1)
-		(end 133 127)
+		(start 147.06 112.12)
+		(end 149 114.06)
 		(width 1)
 		(layer "F.Cu")
@@
 	)
 	(segment
-		(start 135.5 129)
-		(end 136.5 130)
-		(width 1)
-		(layer "F.Cu")
-		(net 0)
-	)
-	(segment
 		(start 150 146.5)
 		(end 150 146)
@@
 	)
 	(segment
-		(start 147.5 130)
-		(end 148 129.5)
-		(width 1)
-		(layer "F.Cu")
-		(net 0)
-	)
-	(segment
 		(start 130.5 60)
 		(end 131.5 59)
@@
 	)
 	(segment
-		(start 133 127)
-		(end 133 130)
-		(width 1)
-		(layer "F.Cu")
-		(net 0)
-	)
-	(segment
 		(start 157.5 134.5)
 		(end 162.5 134.5)
@@
 	)
 	(segment
-		(start 126 124.1)
-		(end 130.1 124.1)
-		(width 1)
-		(layer "F.Cu")
-		(net 0)
-	)
-	(segment
 		(start 118 148)
 		(end 121.06 151.06)
@@
 	)
 	(segment
-		(start 145 112.12)
-		(end 148.06 112.12)
-		(width 0.2)
-		(layer "F.Cu")
-		(net 0)
-	)
-	(segment
 		(start 128.5 98)
 		(end 131 100.5)
@@
 	)
 	(segment
-		(start 176.8 101.76)
-		(end 173 105.56)
-		(width 0.2)
+		(start 126 124.1)
+		(end 130.1 124.1)
+		(width 1)
 		(layer "F.Cu")
 		(net 0)
@@
 	)
 	(segment
-		(start 136.5 130)
-		(end 147.5 130)
-		(width 1)
-		(layer "F.Cu")
-		(net 0)
-	)
-	(segment
 		(start 117.8 61.56)
 		(end 117.8 72.38)
@@
 	)
 	(segment
+		(start 136.5 130)
+		(end 146.5 130)
+		(width 1)
+		(layer "F.Cu")
+		(net 0)
+	)
+	(segment
 		(start 152.825002 69.674998)
 		(end 152.825002 61.335002)
@@
 	)
 	(segment
+		(start 131.06 121.56)
+		(end 135.5 126)
+		(width 1)
+		(layer "F.Cu")
+		(net 0)
+	)
+	(segment
 		(start 169.5 113.5)
 		(end 170 113.5)
@@
 	)
 	(segment
+		(start 145 112.12)
+		(end 147.06 112.12)
+		(width 1)
+		(layer "F.Cu")
+		(net 0)
+	)
+	(segment
 		(start 169 143.56)
 		(end 148.5 143.56)
@@
 	)
 	(segment
+		(start 130.1 124.1)
+		(end 133 127)
+		(width 1)
+		(layer "F.Cu")
+		(net 0)
+	)
+	(segment
 		(start 142.46 109.58)
 		(end 143.88 111)
@@
 	)
 	(segment
+		(start 146.74 119.74)
+		(end 147 120)
+		(width 1)
+		(layer "F.Cu")
+		(net 0)
+	)
+	(segment
 		(start 154 120)
 		(end 155 121)
@@
 	)
 	(segment
+		(start 149 132.5)
+		(end 151 130.5)
+		(width 1)
+		(layer "F.Cu")
+		(net 0)
+	)
+	(segment
 		(start 134.02 90.5)
 		(end 138 90.5)
@@
 	)
 	(segment
+		(start 146.5 130)
+		(end 149 127.5)
+		(width 1)
+		(layer "F.Cu")
+		(net 0)
+	)
+	(segment
 		(start 122 90)
 		(end 123.5 88.5)
@@
 	)
 	(segment
-		(start 133 130)
-		(end 135.5 132.5)
-		(width 1)
-		(layer "F.Cu")
-		(net 0)
-	)
-	(segment
-		(start 135.5 126)
-		(end 135.5 129)
-		(width 1)
-		(layer "F.Cu")
-		(net 0)
-	)
-	(segment
 		(start 149.5 148.06)
 		(end 149.5 147)
@@
 	)
 	(segment
-		(start 147.78 122.28)
-		(end 148 122.5)
+		(start 133 127)
+		(end 133 130)
+		(width 1)
+		(layer "F.Cu")
+		(net 0)
+	)
+	(segment
+		(start 126 121.56)
+		(end 131.06 121.56)
 		(width 1)
 		(layer "F.Cu")
@@
 	)
 	(segment
-		(start 135.5 132.5)
-		(end 149 132.5)
+		(start 149 127.5)
+		(end 149 114.06)
 		(width 1)
 		(layer "F.Cu")
@@
 	)
 	(segment
-		(start 147.74 119.74)
-		(end 148 120)
+		(start 151 112.5)
+		(end 150.5 112)
 		(width 1)
 		(layer "F.Cu")
@@
 	)
 	(segment
-		(start 177 100.56)
-		(end 172 105.56)
-		(width 0.2)
-		(layer "F.Cu")
-		(net 0)
-	)
-	(segment
 		(start 138.94 150)
 		(end 138.825002 149.885002)
@@
 	)
 	(segment
+		(start 151 130.5)
+		(end 151 112.5)
+		(width 1)
+		(layer "F.Cu")
+		(net 0)
+	)
+	(segment
 		(start 139.5 127.56)
 		(end 140.5 128.56)
@@
 	)
 	(segment
+		(start 133 130)
+		(end 135.5 132.5)
+		(width 1)
+		(layer "F.Cu")
+		(net 0)
+	)
+	(segment
 		(start 128.5 133)
 		(end 130 131.5)
@@
 		(width 1)
 		(layer "F.Cu")
+		(net 0)
+	)
+	(segment
+		(start 145 122.28)
+		(end 146.78 122.28)
+		(width 1)
+		(layer "F.Cu")

Commit message: [2026-03-13 14:48:15 From Windows 11 Home]: Windows auto commit
Parts:
- added ?: , , F.Cu at (173.5, 99.5)
- added ?: , , F.Cu at (144.0, 140.0)
- added ?: , , F.Cu at (177.5, 96.0)
- added ?: , , F.Cu at (123.0, 100.5)
- added ?: , , F.Cu at (139.0, 140.0)
- added ?: , , F.Cu at (128.5, 100.5)
- moved ? 1.12 mm to (153.5, 140.5)
- moved ? 1.00 mm to (149.5, 134.5)
- moved ? 1.00 mm to (149.5, 137.5)
- moved ? 1.00 mm to (150.0, 140.5)
Routing:
- net (no net): track 1047.0 -> 1015.7 mm

Commit message: [2026-03-13 15:18:16 From Windows 11 Home]: Windows auto commit
Parts:
- added ?: , , F.Cu at (147.5, 142.5)
- added ?: , , F.Cu at (142.5, 89.1)
- added ?: , , F.Cu at (142.4, 86.5)
- moved ? 0.50 mm to (123.5, 100.5)
Routing:
- net (no net): track 1015.7 -> 1046.2 mm

Commit message: [2026-03-14 00:01:56 From Windows 11 Home]: Windows auto commit
Parts:
- added ?: , , F.Cu at (175.8, 91.4)
- added ?: , , F.Cu at (176.3, 84.8)
- moved REF** 0.34 mm to (147.3, 119.9)
- moved REF** 0.33 mm to (147.3, 122.4)
Routing:
- net (no net): track 1046.2 -> 1042.3 mm
