File: Design/circuit design/circuit design.kicad_pcb (KiCad board)
At the start: 2 copper layers, 18 parts, among them K1 R2_1A05, U1 STM32H7xx Dev Board, U2 ESP-01S, U3 HM-10, U4 uBlox_NEO_7M, U5 E-Paper_296x152_SSD1680, U6 MP1584EN, U7 EasyCard_IC, U8 TP4056

Commit message: [2026-03-13 15:18:16 From Windows 11 Home]: Windows auto commit
Parts:
- removed the REF** at (103.5, 152.0)
- removed the REF** at (100.5, 130.5)
- removed the REF** at (100.5, 151.9)
- removed the REF** at (101.5, 144.0)
- removed the REF** at (100.5, 127.5)
- removed the REF** at (101.5, 147.0)
- removed the REF** at (123.0, 119.5)
- removed the REF** at (122.9, 116.5)
- added ?: , , F.Cu at (173.5, 99.5)
- added ?: , , F.Cu at (153.0, 146.0)
- added ?: , , F.Cu at (144.0, 140.0)
- added ?: , , F.Cu at (149.5, 134.5)
- added ?: , , F.Cu at (149.5, 137.5)
- added ?: , , F.Cu at (177.5, 96.0)
- added ?: , , F.Cu at (176.0, 117.5)
- added ?: , , F.Cu at (123.0, 100.5)
- added ?: , , F.Cu at (170.0, 117.5)
- added ?: , , F.Cu at (147.0, 142.5)
- added ?: , , F.Cu at (150.0, 140.5)
- added ?: , , F.Cu at (139.0, 140.0)
- added ?: , , F.Cu at (170.0, 113.5)
- added ?: , , F.Cu at (128.5, 100.5)
- added ?: , , F.Cu at (153.5, 140.5)
- added ?: , , F.Cu at (176.0, 113.5)
- added ?: , , F.Cu at (150.0, 146.0)
- added REF**: TestPoint_Pad_D1.0mm, TestPoint:TestPoint_Pad_D1.0mm, F.Cu at (157.5, 134.5)
- added REF**: TestPoint_Pad_D1.0mm, TestPoint:TestPoint_Pad_D1.0mm, F.Cu at (147.0, 120.0)
- added REF**: TestPoint_Pad_D1.0mm, TestPoint:TestPoint_Pad_D1.0mm, F.Cu at (147.0, 122.5)
- added REF**: TestPoint_Pad_D1.0mm, TestPoint:TestPoint_Pad_D1.0mm, F.Cu at (153.0, 120.0)
- added REF**: TestPoint_Pad_D1.0mm, TestPoint:TestPoint_Pad_D1.0mm, F.Cu at (157.5, 137.5)
- added REF**: TestPoint_Pad_D1.0mm, TestPoint:TestPoint_Pad_D1.0mm, F.Cu at (153.0, 122.5)
- U1: footprint Module:MODULE_STM327H7xx Dev Module -> Module:MODULE_STM327H7xx Dev Module_1
- U2: footprint Connector_PinHeader_2.54mm:PinHeader_2x04_P2.54mm_Vertical -> Module:MODULE_ESP-01
- moved U2 54.6 mm to (128.5, 90.0), turned to 180 degrees
- moved L1 50.1 mm to (130.0, 72.6)
- moved U1 50.1 mm to (161.8, 114.7)
- moved U3 50.1 mm to (136.8, 105.5)
- moved U5 50.1 mm to (156.6, 148.8)
- moved K1 50.1 mm to (117.8, 61.6)
- moved U4 50.1 mm to (126.0, 129.2)
- moved U7 50.1 mm to (123.1, 72.6)
- moved U8 50.1 mm to (138.9, 51.7)
- moved U6 50.1 mm to (163.2, 55.3)
Routing:
- net (no net): track 1096.7 -> 1048.5 mm

Commit message: [2026-03-14 00:18:20 From Windows 11 Home]: Windows auto commit
Parts:
- added ?: , , F.Cu at (142.4, 86.5)
- added ?: , , F.Cu at (175.8, 91.4)
- added ?: , , F.Cu at (176.3, 84.8)
- added ?: , , F.Cu at (142.5, 89.1)
- moved ? 0.50 mm to (147.5, 142.5)
- moved ? 0.50 mm to (123.5, 100.5)
- moved REF** 0.34 mm to (147.3, 119.9)
- moved REF** 0.33 mm to (147.3, 122.4)
Routing:
- net (no net): track 1048.5 -> 1042.3 mm
