File: Design/circuit design/circuit design.kicad_pcb (KiCad board)
At the start: 2 copper layers, 37 parts, among them K1 R2_1A05, U1 STM32H7xx Dev Board, U2 ESP-01S, U3 HM-10, U4 uBlox_NEO_7M, U5 E-Paper_296x152_SSD1680, U6 MP1584EN, U7 EasyCard_IC, U8 TP4056

Commit message: [2026-03-20 10:18:17 From Windows 11 Home]: Windows auto commit
Routing:
- net (no net): track 1042.3 -> 1044.6 mm
Other:
- board text added: "If you see this then the warranty is void"
- board text removed: "If you see this then warrenty void"

Commit message: [2026-03-27 11:18:17 From Windows 11 Home]: Windows auto commit
Parts:
- added ? (x2): , , F.Cu at (128.5, 92.7)
- added ?: , , F.Cu at (123.2, 76.5)
- added ? (x2): , , F.Cu at (128.5, 97.8)
- added ?: , , F.Cu at (130.6, 76.5)
- moved L1 3.08 mm to (133.1, 72.6)
- moved ? 0.84 mm to (169.2, 117.5)
- moved ? 0.84 mm to (169.2, 113.5)
- moved ? 0.56 mm to (122.9, 100.5)
- moved ? 0.53 mm to (129.0, 100.5)
Routing:
- net (no net): track 1044.6 -> 1046.7 mm
Other:
- board text added: "v1.2.0"
- board text removed: "v1.0.0"

Commit message: [2026-03-27 17:41:40 From Windows 11 Home]: Windows auto commit
Other:
- board text added: "v1.2.1"
- board text removed: "v1.2.0"
Changed lines of the file:
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@@
 		)
 	)
-	(gr_text "v1.2.0\n"
+	(gr_text "v1.2.1"
 		(at 173.482 150.368 0)
 		(layer "User.1")
