File: Design/circuit design/New folder/circuit design.kicad_pcb (KiCad board)
At the start: 2 copper layers, 16 parts, among them K1 R2_1A05, U1 STM32H7xx Dev Board, U2 ESP-01S, U3 HM-10, U4 uBlox_NEO_7M, U5 E-Paper_296x152_SSD1680, U6 MP1584EN, U7 EasyCard_IC, U8 TP4056

Commit message: [2026-03-13 10:48:16 From Windows 11 Home]: Windows auto commit
Parts:
- removed the REF** at (153.0, 137.5)
- removed the REF** at (153.0, 135.0)
- added REF**: L_1206_3216Metric, Inductor_SMD:L_1206_3216Metric, F.Cu at (100.5, 130.5)
- added REF**: L_1206_3216Metric, Inductor_SMD:L_1206_3216Metric, F.Cu at (101.5, 144.0)
- added REF**: L_1206_3216Metric, Inductor_SMD:L_1206_3216Metric, F.Cu at (100.5, 127.5)
- added REF**: L_1206_3216Metric, Inductor_SMD:L_1206_3216Metric, F.Cu at (101.5, 147.0)
- moved L1 50.1 mm to (80.5, 80.5)
- moved REF** 50.1 mm to (122.9, 116.5)
- moved U1 50.1 mm to (112.3, 122.6)
- moved U3 50.1 mm to (87.3, 113.5)
- moved U5 50.1 mm to (107.1, 156.8)
- moved K1 50.1 mm to (68.3, 69.5)
- moved REF** 50.1 mm to (103.5, 152.0)
- moved REF** 50.1 mm to (100.5, 151.9)
- moved REF** 50.1 mm to (123.0, 119.5)
- moved U2 50.1 mm to (78.4, 111.7)
- moved U4 50.1 mm to (76.5, 137.1)
- moved U7 50.1 mm to (73.6, 80.5)
- moved U8 50.1 mm to (89.4, 59.6)
- moved U6 50.1 mm to (113.7, 63.3)
Routing:
- net (no net): track 1053.6 -> 1096.7 mm
